Commit message: Update my_robot.xacro

File: my_robot/urdf/my_robot.xacro (robot description, xacro)
@@ -100,5 +100,5 @@
       </visual>
     </link>
-       <joint name="right_wheel_hinge" type="continous" >
+       <joint name="right_wheel_hinge" type="continuous" >
         <origin xyz="0 -0.125 0" rpy="0 0 0"/>
         <child link="right_wheel"/>
@@ -108,5 +108,5 @@
         <dynamics damping="1.0" friction="1.0"/>
        </joint>
-       <joint name="left_wheel_hinge" type="continous">
+       <joint name="left_wheel_hinge" type="continuous">
         <origin xyz="0 0.125 0" rpy="0 0 0"/>
         <child link="left_wheel"/>

Commit message: Update my_robot.xacro

File: my_robot/urdf/my_robot.xacro (robot description, xacro)
@@ -170,3 +170,15 @@
        <child link="hokuyo"/>
      </joint>
+    <gazebo reference="chassis">
+      <material>Gazebo/Green</material>
+    </gazebo>
+    <gazebo reference="right-wheel">
+      <material>Gazebo/Black</material>
+    </gazebo>
+    <gazebo reference="left_wheel">
+      <material>Gazebo/Black</material>
+    </gazebo>
+    <gazebo reference="camera">
+     <material>Gazebo/white</material>
+    </gazebo>
 </robot>

Commit message: Update my_robot.xacro

File: my_robot/urdf/my_robot.xacro (robot description, xacro)
@@ -104,5 +104,5 @@
         <child link="right_wheel"/>
         <parent link="chassis"/>
-        <axis type="0 -1 0" rpy="0 0 0" />
+        <axis type="0 1 0" rpy="0 0 0" />
         <limit effort="10000" velocity="1000"/>
         <dynamics damping="1.0" friction="1.0"/>

Commit message: Update my_robot.xacro

File: my_robot/urdf/my_robot.xacro (robot description, xacro)
@@ -8,5 +8,5 @@
       <child link="chassis"/>
     </joint>
-    <link name='chassis'>
+    <link name="chassis">
      <pose>0 0 0.1 0 0 0</pose>
      <inertial>
@@ -56,5 +56,5 @@
      </visual>
     </link>
-   <link name='left_wheel'>
+   <link name="left_wheel">
       <inertial>
       <origin xyz="0 0 0" rpy="0 1.5707 1.5707"/>
@@ -100,5 +100,5 @@
       </visual>
     </link>
-       <joint name="right_wheel_hinge" type="continuous" >
+       <joint name="right_wheel_hinge" type="continuous">
         <origin xyz="0 -0.125 0" rpy="0 0 0"/>
         <child link="right_wheel"/>

Commit message: Update my_robot.xacro

File: my_robot/urdf/my_robot.xacro (robot description, xacro)
@@ -8,5 +8,5 @@
       <child link="chassis"/>
     </joint>
-    <link name="chassis">
+    <link name='chassis'>
      <pose>0 0 0.1 0 0 0</pose>
      <inertial>

Commit message: Update my_robot.xacro

File: my_robot/urdf/my_robot.xacro (robot description, xacro)
@@ -104,5 +104,5 @@
         <child link="right_wheel"/>
         <parent link="chassis"/>
-        <axis type="0 1 0" rpy="0 0 0" />
+        <axis xyz="0 1 0" rpy="0 0 0" />
         <limit effort="10000" velocity="1000"/>
         <dynamics damping="1.0" friction="1.0"/>
@@ -112,5 +112,5 @@
         <child link="left_wheel"/>
         <parent link="chassis"/>
-        <axis type="0 1 0" rpy="0 0 0" />
+        <axis xyz="0 1 0" rpy="0 0 0" />
         <limit effort="10000" velocity="1000"/>
         <dynamics damping="1.0" friction="1.0"/>
